File: smart-meter-interface.kicad_sch (KiCad schematic)
At the start: 35 parts, among them J1 USB_B_Micro, Q1 PT26-21B/TR8, Q2 AO3400A, Q3 UMH3N, U2 ESP32-WROOM-32, U3 74LVC1G17DBVR, U4 CH340C

Commit message: Refactor to use Comperator instead of Schmitt Trigger
Parts:
- removed JP2: BOOT, Jumper:SolderJumper-2_P1.3mm_Open_RoundedPad1.0x1.5mm, symbol Jumper:SolderJumper_2_Open
- removed Q2: AO3400A, Package_TO_SOT_SMD:SOT-23, symbol eHZ-Serial-rescue:BSS138-transistors
- removed Q3: UMH3N, Package_TO_SOT_SMD:SOT-363_SC-70-6, symbol Transistor_BJT:UMH3N
- removed R2, R3: 1K, Resistor_SMD:R_0402_1005Metric, symbol Device:R
- removed U3: 74LVC1G17DBVR, Package_TO_SOT_SMD:SOT-23-5, symbol 74xGxx:74LVC1G17
- added D5: LED, LED_SMD:LED_0603_1608Metric, symbol Device:LED
- added Q2, Q3: 2N7002, Package_TO_SOT_SMD:SOT-23, symbol Transistor_FET:2N7002
- added R12: 12k, Resistor_SMD:R_0402_1005Metric, symbol eHZ-Serial-rescue:R-device
- added R13, R15: 1k, Resistor_SMD:R_0402_1005Metric, symbol eHZ-Serial-rescue:R-device
- added R14: 10k, Resistor_SMD:R_0402_1005Metric, symbol eHZ-Serial-rescue:R-device
- added SW1: BOOT, LCSC:KEY-SMD_SKTGLBE010, symbol Switch:SW_Push
- added SW2: RESET, LCSC:KEY-SMD_SKTGLBE010, symbol Switch:SW_Push
- added TP1, TP10, TP11, TP2, TP3, TP4, TP5, TP6, TP7, TP8, TP9: TestPoint_Small, TestPoint:TestPoint_Pad_D1.0mm, symbol Connector:TestPoint_Small
- added U3: MCP6541T-I/OT, Package_TO_SOT_SMD:SOT-23-5, symbol Comparator:MCP6561-OT
- D1: value IR26-21C/L110/CT -> XL-2012IRC-940; footprint LED_SMD:LED_1206_3216Metric -> LCSC:LED0805-RD; LCSC C131280 -> C965889
- JP1: value RESET -> SolderJumper_2_Open
- Q1: value PT26-21B/TR8 -> PT17-21C/L41/TR8; footprint LED_SMD:LED_1206_3216Metric -> LCSC:OPTO-SMD_L2.0-W1.3-R-FD; LCSC C131248 -> C100090
- R1: value 10k -> 1k; LCSC C25744 -> C11702
Connections:
- net +3V3: now also R12.1, R15.1, TP5.1, U3.5 (V+)
- net +5V: now also TP4.1
- net BLINK: now also Q2.1 (G), TP3.1
- net EN: now also TP9.1
- net GND: now also Q2.2 (S), Q3.2 (S), R13.2, R14.2, SW1.1, SW2.1, TP11.1, U3.2 (V-); no longer JP1.1 (A)
- net IO0: now also TP8.1
- net RX: now also JP1.1 (A), TP1.1, U3.1
- net RXD0: now also TP6.1
- net TXD0: now also TP7.1
- net at D1.1 (K): now also Q2.3 (D)
- net at Q1.1 (C), R1.2: now also TP2.1, U3.4 (-)
- net at JP1.2 (B): now also Q3.1 (G), R14.1, TP10.1; no longer R10.1
- net at R11.1: now also SW2.2
- new net: D5.1 (K), Q3.3 (D)
- new net: D5.2 (A), R15.2
- new net: R10.1, SW1.2
- new net: R12.2, R13.1, U3.3 (+)
Other:
- note added: "BOOT / RESET Buttons"
- note removed: "AUTO RESET"
- note removed: "RESET / BOOT"
- moved on the sheet: C10, C9, R10, R11, R6, R7

Commit message: Final adjustments, next prototypes are ordered
Parts:
- removed TP10, TP8, TP9: TestPoint_Small, TestPoint:TestPoint_Pad_D1.0mm, symbol Connector:TestPoint_Small
- added JP2: SolderJumper_2_Open, Jumper:SolderJumper-2_P1.3mm_Open_RoundedPad1.0x1.5mm, symbol Jumper:SolderJumper_2_Open
- added R16: 12k, Resistor_SMD:R_0402_1005Metric, symbol eHZ-Serial-rescue:R-device
- added TP12: TestPoint_Small, TestPoint:TestPoint_Pad_D1.0mm, symbol Connector:TestPoint_Small
Connections:
- net GND: now also TP12.1
- net RX: now also R16.2
- net at R12.2, R13.1, U3.3 (+): now also JP2.1 (A)
- new net: JP2.2 (B), R16.1
Other:
- moved on the sheet: TP11

Commit message: Major cleanup, hopefully working prototype orderd
Parts:
- removed D5: LED, LED_SMD:LED_0603_1608Metric, symbol Device:LED
- removed JP1, JP2: SolderJumper_2_Open, Jumper:SolderJumper-2_P1.3mm_Open_RoundedPad1.0x1.5mm, symbol Jumper:SolderJumper_2_Open
- removed Q3: 2N7002, Package_TO_SOT_SMD:SOT-23, symbol Transistor_FET:2N7002
- removed R14: 10k, Resistor_SMD:R_0402_1005Metric, symbol eHZ-Serial-rescue:R-device
- removed R15: 1k, Resistor_SMD:R_0402_1005Metric, symbol eHZ-Serial-rescue:R-device
- removed SW1: BOOT, LCSC:KEY-SMD_SKTGLBE010, symbol Switch:SW_Push
- removed SW2: RESET, LCSC:KEY-SMD_SKTGLBE010, symbol Switch:SW_Push
- removed U4: CH340C, Package_SO:SOIC-16_3.9x9.9mm_P1.27mm, symbol Interface_USB:CH340C
- added SW1: BOOT, LCSC:SW-SMD_4P-L5.1-W5.1-P3.70-LS6.5-TL-2, symbol Switch:SW_MEC_5E
- added SW2: RESET, LCSC:SW-SMD_4P-L5.1-W5.1-P3.70-LS6.5-TL-2, symbol Switch:SW_MEC_5E
- added U1: CH340E, Package_SO:MSOP-10_3x3mm_P0.5mm, symbol Interface_USB:CH340E
- R1: value 1k -> 10k
- R16: value 12k -> 12k DNP; now not fitted; now left out of the parts list
Connections:
- net +5V: now also U1.7 (VCC)
- net D+: now also U1.1 (UD+)
- net D-: now also U1.2 (UD-)
- net GND: now also SW1.3 (K), SW1.4 (A), SW2.3 (K), SW2.4 (A), U1.3 (GND)
- net RXD0: now also U1.8 (TXD)
- net TXD0: now also U1.9 (RXD)
- net at Q1.1 (C), R1.2, TP2.1: now also R16.1, U3.3 (+); no longer U3.4 (-)
- net at C1.2: now also U1.10 (V3)
- net at R10.1: now also SW1.1, SW1.2
- net at R11.1: now also SW2.1, SW2.2
- net at R12.2, R13.1: now also U3.4 (-); no longer U3.3 (+)
Other:
- moved on the sheet: TP2

Commit message: Fixed wrong LCSC number of R1
Parts:
- R1: LCSC C11702 -> C25744
Changed lines of the file:
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@@
       (effects (font (size 1.27 1.27)) hide)
     )
-    (property "LCSC" "C11702" (at 32.385 41.91 0)
+    (property "LCSC" "C25744" (at 32.385 41.91 0)
       (effects (font (size 1.27 1.27)) hide)
     )
