File: kicad/smart-meter-interface.kicad_pcb (KiCad board)
At the start: 2 copper layers, 32 x 32 mm, 52 parts, among them J1 USB_B_Micro, Q1 PT17-21C/L41/TR8, Q2 2N7002, SW1 BOOT, SW2 RESET, U1 CH340E, U2 ESP32-WROOM-32, U3 MCP6541T-I/OT

Commit message: Minor cleanups for V1.1
Parts:
- removed R16: 12k DNP, Resistor_SMD:R_0402_1005Metric
- removed the TP1 at (67.7, 60.4)
- removed TP11, TP6, TP7: TestPoint_Small, TestPoint:TestPoint_Pad_D1.0mm
- removed the TP2 at (67.7, 50.3)
- removed the TP3 at (67.7, 57.9)
- removed kibuzzard-635BBB3D: G***, kibuzzard-635BBB3D
- removed kibuzzard-635BBB71: G***, kibuzzard-635BBB71
- added kibuzzard-63C57633: G***, kibuzzard-63C57633, F.Cu at (56.2, 67.6)
- added kibuzzard-63C57836: G***, kibuzzard-63C57836, F.Cu at (70.3, 56.1)
- TP1: renamed from TP12; moved to B.Cu
- TP2: renamed from TP4; moved to B.Cu
- TP3: renamed from TP5; moved to B.Cu
- moved TP2 6.83 mm to (41.6, 58.8), turned to 180 degrees
- moved TP1 4.26 mm to (41.6, 47.8), turned to 180 degrees
- moved TH1 0.71 mm to (42.0, 42.0)
- moved TH2 0.71 mm to (70.0, 70.0)
- moved kibuzzard-635BBB9A 0.50 mm to (70.4, 67.4)
- moved kibuzzard-635BBBA9 0.50 mm to (41.6, 67.3)
- turned TP3 to 180 degrees
Routing:
- net Net-(Q1-C): track 18.6 -> 9.90 mm, vias 3 -> 0
- net RX: track 26.3 -> 18.4 mm, vias 3 -> 1
- net +5V: track 27.6 -> 22.9 mm
- net RXD0: track 26.5 -> 21.8 mm
- net BLINK: track 32.1 -> 27.6 mm
- net TXD0: track 25.9 -> 22.4 mm
- net GND: vias 46 -> 45
Other:
- outline, holes or cut-outs redrawn
- board text removed: "BL"
- board text removed: "Q1"
- board text removed: "RX"
- board text removed: "RxD"
- board text removed: "TxD"

Commit message: Don't know what changed, something minor for sure
Parts:
- removed kibuzzard-63C57633: G***, kibuzzard-63C57633
- added RV1: 20k, lcsc:RES-ADJ-SMD_3P-L3.8-W3.0-P2.00-BL-FS, B.Cu at (55.4, 48.7)
- added TP4: TestPoint_Small, TestPoint:TestPoint_Pad_D1.0mm, F.Cu at (66.9, 47.2)
- added TP5: TestPoint_Small, TestPoint:TestPoint_Pad_D1.0mm, F.Cu at (68.9, 47.2)
- added TP6: TestPoint_Small, TestPoint:TestPoint_Pad_D1.0mm, F.Cu at (71.0, 47.2)
- added kibuzzard-64709697: G***, kibuzzard-64709697, F.Cu at (56.2, 67.6)
- D1: value XL-2012IRC-940 -> LED_W; footprint LCSC:LED0805-RD -> LED_SMD:LED_0805_2012Metric
- D3: value LED -> LED_G
- D4: value LED -> LED_B
- R1: value 10k -> 1k
- TP1: value TestPoint_Small -> TestPoint; footprint TestPoint:TestPoint_Pad_D1.0mm -> TestPoint:TestPoint_Keystone_5000-5004_Miniature; moved to F.Cu
- TP2, TP3: moved to F.Cu
- moved TP2 3.64 mm to (45.2, 59.3), turned to 0 degrees
- moved R1 3.17 mm to (55.4, 51.4), turned to 0 degrees
- moved TP1 2.34 mm to (43.9, 47.3), turned to 0 degrees
- moved TP3 2.24 mm to (45.1, 50.0), turned to 0 degrees
Connections:
- R1 pad 2: Net-(Q1-C) -> Net-(R1-Pad2)
Routing:
- net RX: track 18.4 -> 38.1 mm
- net Net-(Q1-C): track 9.90 -> 22.8 mm, vias 0 -> 1
- net Net-(U3--): track 2.93 -> 9.03 mm, vias 0 -> 1
- net Net-(R1-Pad2): track 0.00 -> 5.69 mm, vias 0 -> 2
- net +3V3: track 58.5 -> 61.1 mm
- net +5V: track 22.9 -> 21.1 mm
- net GND: vias 45 -> 44
Other:
- board text removed: "3V3"
- board text removed: "5V"
- board text removed: "GND"
