File: kicad/smart-meter-interface.kicad_sch (KiCad schematic)
At the start: 44 parts, among them J1 USB_B_Micro, Q1 PT17-21C/L41/TR8, Q2 2N7002, SW1 BOOT, SW2 RESET, U1 CH340E, U2 ESP32-WROOM-32, U3 MCP6541T-I/OT

Commit message: Minor cleanups for V1.1
Parts:
- removed R16: 12k DNP, Resistor_SMD:R_0402_1005Metric, symbol eHZ-Serial-rescue:R-device
- removed TP1, TP11, TP2, TP3, TP6, TP7: TestPoint_Small, TestPoint:TestPoint_Pad_D1.0mm, symbol Connector:TestPoint_Small
- TP1: renamed from TP12; now not fitted; now left out of the parts list
- TP2: renamed from TP4; now not fitted; now left out of the parts list
- TP3: renamed from TP5; now not fitted; now left out of the parts list

Commit message: Don't know what changed, something minor for sure
Parts:
- removed TP1: TestPoint_Small, TestPoint:TestPoint_Pad_D1.0mm, symbol Connector:TestPoint_Small
- added RV1: 20k, lcsc:RES-ADJ-SMD_3P-L3.8-W3.0-P2.00-BL-FS, symbol Device:R_Potentiometer_Small
- added TP1: TestPoint, TestPoint:TestPoint_Keystone_5000-5004_Miniature, symbol Connector:TestPoint
- added TP4, TP5, TP6: TestPoint_Small, TestPoint:TestPoint_Pad_D1.0mm, symbol Connector:TestPoint_Small
- C1, C2, C3, C4, C5, C6, C7, C8, C9, D2: Category (none) -> Basic
- C10: Category (none) -> Basic; LCSC C307331 -> C1523
- D1: value XL-2012IRC-940 -> LED_W; footprint LCSC:LED0805-RD -> LED_SMD:LED_0805_2012Metric; Category (none) -> Basic; LCSC C965889 -> C34499
- D3: value LED -> LED_G; Category (none) -> Basic
- D4: value LED -> LED_B; Category (none) -> Basic
- J1, LDO1: Category (none) -> Extended
- R1: value 10k -> 1k; LCSC C25744 -> C11702
Connections:
- net GND: now also TP1.1
- net RX: now also TP6.1
- net at Q1.1 (C), U3.3 (+): now also RV1.3, TP4.1; no longer R1.2
- net at R12.2, R13.1, U3.4 (-): now also TP5.1
- new net: R1.2, RV1.1, RV1.2
Other:
- moved on the sheet: R1
