File: hardware/smart-meter-interface.kicad_sch (KiCad schematic)
At the start: 31 parts, among them J1 USB_B_Micro, Q3 SFH309, Q4 BC817W, Q5 BC807W, U1 CH340X, U2 ESP32-WROOM-32, U4 74LVC1G17, U5 74LVC1G17

Commit message: Streamlined annotations
Parts:
- renumbered C9 to C1, C7 to C10, C8 to C11, C10 to C2, C11 to C3, C1 to C4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
